File: poe.kicad_pcb (KiCad board)
At the start: 2 copper layers, 15 parts, among them P1 CONN_01X08

Commit message: Stuff… Much Stuff…
(i know this commit is bad… but it would have been necessary ages ago)
Parts:
- removed 1.65k1, 1.65k2: R, Resistors_ThroughHole:Resistor_Horizontal_RM20mm
- removed D10: LED, LEDs:LED-3MM
- added C1: >= 450 µF, Discret:C2V8, F.Cu at (83.0, 53.0)
- added J1: RJ45, Custom:RJ45_8, F.Cu at (123.0, 42.0)
- added Q1: IRF640, pth-semi:TO-220, F.Cu at (106.0, 70.0)
- added R3: 22k, Resistors_ThroughHole:Resistor_Horizontal_RM15mm, F.Cu at (112.0, 55.0)
- added R4: 22k, Resistors_ThroughHole:Resistor_Horizontal_RM15mm, F.Cu at (111.0, 29.0)
- added R5: 3.3k, Resistors_ThroughHole:Resistor_Horizontal_RM15mm, F.Cu at (90.0, 58.0)
- added R6: 3.3k, Resistors_ThroughHole:Resistor_Horizontal_RM15mm, F.Cu at (83.0, 29.0)
- added SW1: Switch_SPDT_x2, Custom:Switch, F.Cu at (107.0, 77.0)
- added U1: Step_Down, Custom:Step-Down, F.Cu at (56.0, 52.0)
- added U2: Bananasocket, Custom:Bananasocket, F.Cu at (76.0, 35.0)
- added U3: Bananasocket, Custom:Bananasocket, F.Cu at (38.0, 35.0)
- added U4: Bananasocket, Custom:Bananasocket, F.Cu at (76.0, 74.0)
- added U5: Bananasocket, Custom:Bananasocket, F.Cu at (38.0, 74.0)
- D1, D2: footprint Diodes_ThroughHole:Diode_DO-35_SOD27_Horizontal_RM10 -> Custom:Diode-Bridge
- D7: value LED -> ZENER; footprint LEDs:LED-3MM -> Discret:D3
- P1: value CONN_01X08 -> USB_A; footprint Pin_Headers:Pin_Header_Angled_1x08 -> Connect:USB_A
- R1, R2: value 22kΩ -> 1M; footprint Resistors_ThroughHole:Resistor_Horizontal_RM7mm -> Resistors_ThroughHole:Resistor_Horizontal_RM15mm
- moved P1 160.4 mm to (63.0, 35.0), turned to 180 degrees
- moved D1 115.4 mm to (100.0, 50.0), turned to 45 degrees
- moved D2 112.2 mm to (100.0, 33.5), turned to 45 degrees
- moved R1 111.3 mm to (108.0, 61.0), turned to 180 degrees
- moved D5 88.1 mm to (97.0, 37.0), turned to 270 degrees
- moved D9 76.9 mm to (90.0, 35.0), turned to 270 degrees
- moved D4 76.8 mm to (97.0, 48.0), turned to 90 degrees
- moved R2 76.2 mm to (93.0, 64.0), turned to 0 degrees
- moved D6 74.1 mm to (94.0, 48.0), turned to 90 degrees
- moved D7 69.3 mm to (94.0, 37.0), turned to 270 degrees
- moved D3 68.0 mm to (87.0, 64.0), turned to 180 degrees
- moved D8 58.6 mm to (90.0, 46.0), turned to 270 degrees
Connections:
- D1 pad 1: Net-(D1-Pad1) -> Ethernet-
- D1 pad 2: Net-(1.65k1-Pad2) -> Net-(D1-Pad2)
- D2 pad 1: Net-(D1-Pad1) -> Ethernet-
- D3 pad 1: Net-(D1-Pad4) -> Ethernet+
- D4 pad 1: Net-(D2-Pad2) -> Net-(D1-Pad4)
- D5 pad 1: Net-(D5-Pad1) -> Net-(D2-Pad2)
- D5 pad 2: Net-(D3-Pad2) -> Net-(D5-Pad2)
- D6 pad 1: Net-(D10-Pad1) -> Net-(D6-Pad1)
- D7 pad 1: Net-(D5-Pad1) -> Net-(D7-Pad1)
- D7 pad 2: Net-(1.65k1-Pad1) -> Net-(D5-Pad2)
- D8 pad 1: Net-(1.65k2-Pad1) -> Net-(D6-Pad1)
- D8 pad 2: Net-(D10-Pad1) -> Net-(D8-Pad2)
- D9 pad 1: Net-(1.65k1-Pad1) -> Net-(D9-Pad1)
- D9 pad 2: Net-(D5-Pad1) -> Net-(D7-Pad1)
- P1 pad 1: Net-(D2-Pad2) -> VDD
- P1 pad 2: Net-(D2-Pad2) -> Net-(P1-Pad2)
- P1 pad 3: Net-(1.65k2-Pad2) -> Net-(P1-Pad2)
- P1 pad 4: Net-(1.65k1-Pad2) -> GND
- P1 pad 5: Net-(1.65k1-Pad2) -> Net-(P1-Pad5)
- R1 pad 1: Net-(D1-Pad4) -> Net-(Q1-Pad1)
- R1 pad 2: Net-(1.65k1-Pad2) -> Ethernet-
- R2 pad 1: Net-(1.65k2-Pad2) -> Net-(D3-Pad2)
- R2 pad 2: Net-(D2-Pad2) -> Net-(Q1-Pad1)
Routing:
- net Ethernet-: track 0.00 -> 67.1 mm
- net Ethernet+: track 0.00 -> 65.7 mm
- net Net-(D1-Pad2): track 0.00 -> 53.7 mm
- net Net-(D1-Pad4): track 95.3 -> 45.5 mm
- net Net-(D2-Pad4): track 0.00 -> 42.7 mm
- net Net-(D2-Pad2): track 29.5 -> 0.00 mm
- net Net-(1.65k1-Pad2): track 21.6 -> 0.00 mm
- net Net-(D1-Pad1): track 20.3 -> 0.00 mm
- net Net-(D9-Pad1): track 0.00 -> 9.49 mm
- net Net-(D8-Pad2): track 0.00 -> 9.46 mm
- net Net-(Q1-Pad1): track 0.00 -> 9.22 mm
- net Net-(D7-Pad1): track 0.00 -> 5.35 mm
- net Net-(D6-Pad1): track 0.00 -> 4.75 mm
- net Net-(D5-Pad2): track 0.00 -> 3.00 mm
- net Net-(D4-Pad2): track 0.00 -> 3.00 mm
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- added copper zone on B.Cu, net GND
- added copper zone on F.Cu, net GND
- added copper zone on F.Cu, net Net-(D2-Pad2)
- added copper zone on F.Cu, net VDD
Other:
- board outline added: 100 x 56 mm
- net class Default: clearance 0.2 -> 0.5; trace_width 0.25 -> 1
- net class Thick added: clearance 1, trace_width 5, via_dia 0.6, via_drill 0.4
- rule trace_clearance: 0.2 -> 0.5
- rule trace_min: 0.2 -> 1
- board text added: "+"
- board text added: "-"
- board text added: "@Ranlvor"
- board text added: "Auto"
- board text added: "Force ON"

Commit message: various unknown changes
Parts:
- added JP1: CONN_02X01, Custom:2-Jumper, F.Cu at (54.0, 65.5)
- added W1: TEST_1P, Custom:1x1cm-SMD-solderpad, F.Cu at (50.0, 75.0)
- added W2: TEST_1P, Custom:1x1cm-SMD-solderpad, F.Cu at (122.0, 70.0)
- moved C1 2.24 mm to (84.0, 55.0)
Connections:
- J1 pad 9: (no net) -> Earth
- P1 pad 5: Net-(P1-Pad5) -> Earth
Routing:
- net Earth: track 0.00 -> 99.8 mm
- net GND: track 0.00 -> 29.3 mm, vias 0 -> 5
- net Net-(D3-Pad2): track 0.00 -> 2.19 mm
- net (no net): vias 1 -> 0
- added copper zone on B.Cu, net Earth
Other:
- board text added: "GND"
- board text added: "VDD"
