File: poe.sch (KiCad schematic (older format))
At the start: 25 parts, among them J1 RJ45, P1 USB_A, Q1 IRF640, SW1 Switch_SPDT_x2, U1 Step_Down, U2 Bananasocket, U3 Bananasocket, U4 Bananasocket, U5 Bananasocket

Commit message: various unknown changes
Parts:
- added JP1: CONN_02X01, Custom:2-Jumper, symbol CONN_02X01
- added W1, W2: TEST_1P, Custom:1x1cm-SMD-solderpad, symbol TEST_1P
- J1: footprint Connect:RJ45_8 -> Custom:RJ45_8
- R1, R2, R3, R4, R5, R6: footprint Resistors_ThroughHole:Resistor_Horizontal_RM7mm -> Resistors_ThroughHole:Resistor_Horizontal_RM15mm
Connections:
- net Earth: now also P1.5 (shield)
- net GND: now also JP1.2 (P2), W2.1
- net VDD: now also JP1.1 (P1), W1.1
Changed lines of the file:
@@
 F 0 "R3" V 5580 3050 50  0000 C CNN
 F 1 "22k" V 5500 3050 50  0000 C CNN
-F 2 "Resistors_ThroughHole:Resistor_Horizontal_RM7mm" V 5430 3050 50  0001 C CNN
+F 2 "Resistors_ThroughHole:Resistor_Horizontal_RM15mm" V 5430 3050 50  0001 C CNN
 F 3 "" H 5500 3050 50  0000 C CNN
 	1    5500 3050
@@
 F 0 "R4" V 5580 3800 50  0000 C CNN
 F 1 "22k" V 5500 3800 50  0000 C CNN
-F 2 "Resistors_ThroughHole:Resistor_Horizontal_RM7mm" V 5430 3800 50  0001 C CNN
+F 2 "Resistors_ThroughHole:Resistor_Horizontal_RM15mm" V 5430 3800 50  0001 C CNN
 F 3 "" H 5500 3800 50  0000 C CNN
 	1    5500 3800
@@
 F 0 "R5" V 5830 3300 50  0000 C CNN
 F 1 "3.3k" V 5750 3300 50  0000 C CNN
-F 2 "Resistors_ThroughHole:Resistor_Horizontal_RM7mm" V 5680 3300 50  0001 C CNN
+F 2 "Resistors_ThroughHole:Resistor_Horizontal_RM15mm" V 5680 3300 50  0001 C CNN
 F 3 "" H 5750 3300 50  0000 C CNN
 	1    5750 3300
@@
 F 0 "R6" V 5830 3600 50  0000 C CNN
 F 1 "3.3k" V 5750 3600 50  0000 C CNN
-F 2 "Resistors_ThroughHole:Resistor_Horizontal_RM7mm" V 5680 3600 50  0001 C CNN
+F 2 "Resistors_ThroughHole:Resistor_Horizontal_RM15mm" V 5680 3600 50  0001 C CNN
 F 3 "" H 5750 3600 50  0000 C CNN
 	1    5750 3600
@@
 F 0 "R1" V 4430 4700 50  0000 C CNN
 F 1 "1M" V 4350 4700 50  0000 C CNN
-F 2 "Resistors_ThroughHole:Resistor_Horizontal_RM7mm" V 4280 4700 50  0001 C CNN
+F 2 "Resistors_ThroughHole:Resistor_Horizontal_RM15mm" V 4280 4700 50  0001 C CNN
 F 3 "" H 4350 4700 50  0000 C CNN
 	1    4350 4700
@@
 F 0 "R2" V 4880 4700 50  0000 C CNN
 F 1 "1M" V 4800 4700 50  0000 C CNN
-F 2 "Resistors_ThroughHole:Resistor_Horizontal_RM7mm" V 4730 4700 50  0001 C CNN
+F 2 "Resistors_ThroughHole:Resistor_Horizontal_RM15mm" V 4730 4700 50  0001 C CNN
 F 3 "" H 4800 4700 50  0000 C CNN
 	1    4800 4700
@@
 F 0 "J1" H 3250 3650 50  0000 C CNN
 F 1 "RJ45" H 2900 3650 50  0000 C CNN
-F 2 "Connect:RJ45_8" H 3050 3150 50  0000 C CNN
+F 2 "Custom:RJ45_8" H 3050 3150 50  0000 C CNN
 F 3 "" H 3050 3150 50  0000 C CNN
 	1    3050 3150
@@
 $EndComp
 $Comp
-L Earth #PWR01
+L Earth #PWR1
 U 1 1 5977EB34
 P 2700 2600
-F 0 "#PWR01" H 2700 2350 50  0001 C CNN
+F 0 "#PWR1" H 2700 2350 50  0001 C CNN
 F 1 "Earth" H 2700 2450 50  0001 C CNN
 F 2 "" H 2700 2600 50  0000 C CNN
@@
 $EndComp
 $Comp
-L GND #PWR02
+L GND #PWR11
 U 1 1 598AFB0D
 P 10100 4500
-F 0 "#PWR02" H 10100 4250 50  0001 C CNN
+F 0 "#PWR11" H 10100 4250 50  0001 C CNN
 F 1 "GND" H 10100 4350 50  0000 C CNN
 F 2 "" H 10100 4500 50  0000 C CNN
@@
 $EndComp
 $Comp
-L GND #PWR03
+L GND #PWR2
 U 1 1 598AFE66
 P 4200 5550
-F 0 "#PWR03" H 4200 5300 50  0001 C CNN
+F 0 "#PWR2" H 4200 5300 50  0001 C CNN
 F 1 "GND" H 4200 5400 50  0000 C CNN
 F 2 "" H 4200 5550 50  0000 C CNN
@@
 $EndComp
 $Comp
-L VDD #PWR04
+L VDD #PWR10
 U 1 1 598B02D1
 P 10100 4200
-F 0 "#PWR04" H 10100 4050 50  0001 C CNN
+F 0 "#PWR10" H 10100 4050 50  0001 C CNN
 F 1 "VDD" H 10100 4350 50  0000 C CNN
 F 2 "" H 10100 4200 50  0000 C CNN
@@
 Ethernet+
 $Comp
-L VDD #PWR05
+L VDD #PWR8
 U 1 1 598B1D22
 P 9250 4300
-F 0 "#PWR05" H 9250 4150 50  0001 C CNN
+F 0 "#PWR8" H 9250 4150 50  0001 C CNN
 F 1 "VDD" H 9250 4450 50  0000 C CNN
 F 2 "" H 9250 4300 50  0000 C CNN
@@
 $EndComp
 $Comp
-L GND #PWR06
+L GND #PWR9
 U 1 1 598B1D7E
 P 9250 4400
-F 0 "#PWR06" H 9250 4150 50  0001 C CNN
+F 0 "#PWR9" H 9250 4150 50  0001 C CNN
 F 1 "GND" H 9250 4250 50  0000 C CNN
 F 2 "" H 9250 4400 50  0000 C CNN
@@
 $EndComp
 $Comp
-L GND #PWR07
+L GND #PWR5
 U 1 1 598B1EC7
 P 7600 4500
-F 0 "#PWR07" H 7600 4250 50  0001 C CNN
+F 0 "#PWR5" H 7600 4250 50  0001 C CNN
 F 1 "GND" H 7600 4350 50  0000 C CNN
 F 2 "" H 7600 4500 50  0000 C CNN
@@
 Text GLabel 4200 4400 0    60   Input ~ 0
 Ethernet-
+$Comp
+L GND #PWR7
+U 1 1 59901F81
+P 8250 5650
+F 0 "#PWR7" H 8250 5400 50  0001 C CNN
+F 1 "GND" H 8250 5500 50  0000 C CNN
+F 2 "" H 8250 5650 50  0000 C CNN
+F 3 "" H 8250 5650 50  0000 C CNN
+	1    8250 5650
+	1    0    0    -1
+$EndComp
+$Comp
+L VDD #PWR6
+U 1 1 59901FC9
+P 8250 5150
+F 0 "#PWR6" H 8250 5000 50  0001 C CNN
+F 1 "VDD" H 8250 5300 50  0000 C CNN
+F 2 "" H 8250 5150 50  0000 C CNN
+F 3 "" H 8250 5150 50  0000 C CNN
+	1    8250 5150
+	1    0    0    -1
+$EndComp
+$Comp
+L Earth #PWR12
+U 1 1 599036D7
+P 10500 4700
+F 0 "#PWR12" H 10500 4450 50  0001 C CNN
+F 1 "Earth" H 10500 4550 50  0001 C CNN
+F 2 "" H 10500 4700 50  0000 C CNN
+F 3 "" H 10500 4700 50  0000 C CNN
+	1    10500 4700
+	1    0    0    -1
+$EndComp
+$Comp
+L CONN_02X01 JP1
+U 1 1 59904033
+P 8250 5400
+F 0 "JP1" H 8250 5500 50  0000 C CNN
+F 1 "CONN_02X01" H 8250 5300 50  0000 C CNN
+F 2 "Custom:2-Jumper" H 8250 4200 50  0001 C CNN
+F 3 "" H 8250 4200 50  0000 C CNN
+	1    8250 5400
+	0    1    1    0
+$EndComp
+$Comp
+L TEST_1P W1
+U 1 1 59904467
+P 7300 5200
+F 0 "W1" H 7300 5470 50  0000 C CNN
+F 1 "TEST_1P" H 7300 5400 50  0000 C CNN
+F 2 "Custom:1x1cm-SMD-solderpad" H 7500 5200 50  0001 C CNN
+F 3 "" H 7500 5200 50  0000 C CNN
+	1    7300 5200
+	-1   0    0    1
+$EndComp
+$Comp
+L TEST_1P W2
+U 1 1 599044EF
+P 7300 5850
+F 0 "W2" H 7300 6120 50  0000 C CNN
+F 1 "TEST_1P" H 7300 6050 50  0000 C CNN
+F 2 "Custom:1x1cm-SMD-solderpad" H 7500 5850 50  0001 C CNN
+F 3 "" H 7500 5850 50  0000 C CNN
+	1    7300 5850
+	1    0    0    -1
+$EndComp
+$Comp
+L GND #PWR4
+U 1 1 59904588
+P 7300 5850
+F 0 "#PWR4" H 7300 5600 50  0001 C CNN
+F 1 "GND" H 7300 5700 50  0000 C CNN
+F 2 "" H 7300 5850 50  0000 C CNN
+F 3 "" H 7300 5850 50  0000 C CNN
+	1    7300 5850
+	1    0    0    -1
+$EndComp
+$Comp
+L VDD #PWR3
+U 1 1 599045F0
+P 7300 5200
+F 0 "#PWR3" H 7300 5050 50  0001 C CNN
+F 1 "VDD" H 7300 5350 50  0000 C CNN
+F 2 "" H 7300 5200 50  0000 C CNN
+F 3 "" H 7300 5200 50  0000 C CNN
+	1    7300 5200
+	1    0    0    -1
+$EndComp
 $EndSCHEMATC
